File: Schematics/Eagle/doogie_board.brd (EAGLE design)
At the start: 239.3 x 151.4 mm, 41 parts, among them J1 3.7V, Q1 TEFT4300, Q2 TEFT4300, Q3 TEFT4300, Q4 TEFT4300, Q5 BSS123, Q6 BSS123, Q7 BSS123, Q9 BSS123

Commit message: Remove unnecessary stuffs
Parts:
- removed BUZZER: EMB15, buzzer:BMT1205XH7.5
- removed C13, C15, C17: 10u, rcl:C0805
- removed C14, C16, C18: 0.1u, rcl:C0603
- removed D6: 1SS404, diode:SOD323-R
- removed Q5, Q6, Q7, Q9: BSS123, transistor-small-signal:SOT23
- removed R27: 100k, rcl:R0603
- removed X1, X2: (no value), pololu:PIN4-1
- added T1, T2, T3: BC337, transistor:TO92
- added U$2, U$3, U$4: FRAME_A4P, doogie:FRAME_A4P
- D4: value SFH4545 -> SFH4545KA
- R10, R12, R4, R5, R6, R7, R8: device rcl:R0603 -> rcl:0204/7
- R11, R13, R9: device rcl:R0805 -> rcl:0204/7
- moved U$1 169.8 mm to (85.1, 14.2)
- moved R12 38.3 mm to (-6.67, 40.4)
- moved R6 20.9 mm to (22.4, 37.2), turned to 180 degrees
- moved R7 12.7 mm to (27.0, 51.6)
- moved R4 12.3 mm to (-18.7, 45.9), turned to 90 degrees
- moved R8 10.1 mm to (-21.9, 37.4)
- moved Q1 9.70 mm to (-32.1, 47.8)
- moved Q4 9.70 mm to (32.1, 47.8)
- moved D1 9.70 mm to (-37.2, 40.1)
- moved D4 9.70 mm to (37.2, 40.1)
- moved MOTORS 9.65 mm to (-28.1, -21.6)
- moved R9 9.06 mm to (-32.0, 37.3)
- moved R10 8.96 mm to (3.17, 40.5)
- moved R13 8.90 mm to (32.1, 37.2)
- moved R11 7.61 mm to (6.73, 52.3), turned to 180 degrees
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Connections:
- removed net +3V3: BUZZER.+, C13.1, C14.1, C15.1, C16.1, C17.1, C18.1, D1.A, D2.A, D4.A, D6.C, X1.4, X2.4
- removed net ALT1: X1.2
- removed net ALT2: X2.2
- removed net ALTERNATE_EN: X1.3, X2.3
- removed net A_VDD: Q1.C, Q2.C, Q3.C, Q4.C
- removed net BUZZER: Q9.1, R27.2
- new net N$6: R10.1, T2.2
- new net N$7: R12.1, T3.2
- net 3.3V: now also D1.A, D2.A, D4.A, Q1.C, Q2.C, Q3.C, Q4.C
- net GND: now also T1.1, T2.1, T3.1; no longer C13.2, C14.2, C15.2, C16.2, C17.2, C18.2, Q5.2, Q6.2, Q7.2, Q9.2, R10.1, R12.1, R27.1, R8.1, X1.1, X2.1
- net LF_EMITTER: no longer Q5.1
- net N$1: now also T1.3; no longer Q5.3
- net N$2: now also T2.3; no longer Q6.3
- net N$3: now also T3.3; no longer Q7.3
- net N$4: now also R8.1, T1.2; no longer BUZZER.-, D6.A, Q9.3
- net RF_EMITTER: no longer Q7.1
- net SIDE_EMITTER: no longer Q6.1
Routing:
- net A_VDD: track 99.2 -> 0.00 mm, vias 1 -> 0
- net GND: track 24.6 -> 2.54 mm, vias 6 -> 0
- net +3V3: track 10.1 -> 0.00 mm
- net LF_RECEIVER: track 10.7 -> 1.10 mm
- net N$14: track 8.89 -> 0.00 mm
- net 3.3V: track 3.18 -> 0.00 mm
- net N$16: track 2.65 -> 0.00 mm
- net N$15: track 2.65 -> 0.00 mm
- net N$3: track 2.60 -> 0.00 mm
- net N$1: track 2.60 -> 0.00 mm
- net N$17: track 1.27 -> 0.00 mm
- net N$20: track 0.95 -> 0.00 mm
