File: Schematics/Eagle/doogie_board.sch (EAGLE design)
At the start: 41 parts, among them J1 3.7V, Q1 TEFT4300, Q2 TEFT4300, Q3 TEFT4300, Q4 TEFT4300, Q5 BSS123, Q6 BSS123, Q7 BSS123, Q9 BSS123

Commit message: Remove unnecessary stuffs
Parts:
- removed BUZZER: EMB15, buzzer:BMT1205XH7.5
- removed C13, C15, C17: 10u, rcl:C-EUC0805
- removed C14, C16, C18: 0.1u, rcl:C-EUC0603
- removed D6: 1SS404, diode:DIODE-SOD323-R
- removed Q5, Q6, Q7, Q9: BSS123, transistor-small-signal:BSS123
- removed R27: 100k, rcl:R-EU_R0603
- removed X1, X2: (no value), pololu:MA04-1
- added T1, T2, T3: BC337, transistor:BC337
- added U$2, U$3, U$4: FRAME_A4P, doogie:FRAME_A4P
- D4: value SFH4545 -> SFH4545KA
- R10, R12, R4, R5, R6, R7, R8: device rcl:R-EU_R0603 -> rcl:R-EU_0204/7
- R11, R13, R9: device rcl:R-EU_R0805 -> rcl:R-EU_0204/7
Connections:
- removed net +3V3: BUZZER.+, C13.1, C14.1, C15.1, C16.1, C17.1, C18.1, D1.A, D2.A, D4.A, D6.C, X1.4, X2.4
- removed net ALT1: X1.2
- removed net ALT2: X2.2
- removed net ALTERNATE_EN: X1.3, X2.3
- removed net A_VDD: Q1.C, Q2.C, Q3.C, Q4.C
- removed net BUZZER: Q9.G, R27.2
- new net N$6: R10.1, T2.B
- new net N$7: R12.1, T3.B
- net 3.3V: now also D1.A, D2.A, D4.A, Q1.C, Q2.C, Q3.C, Q4.C
- net GND: now also T1.E, T2.E, T3.E; no longer C13.2, C14.2, C15.2, C16.2, C17.2, C18.2, Q5.S, Q6.S, Q7.S, Q9.S, R10.1, R12.1, R27.1, R8.1, X1.1, X2.1
- net LF_EMITTER: no longer Q5.G
- net N$1: now also T1.C; no longer Q5.D
- net N$2: now also T2.C; no longer Q6.D
- net N$3: now also T3.C; no longer Q7.D
- net N$4: now also R8.1, T1.B; no longer BUZZER.-, D6.A, Q9.D
- net RF_EMITTER: no longer Q7.G
- net SIDE_EMITTER: no longer Q6.G
Other:
- moved on the sheet: D1, D2, D3, D4, Q1, Q2, Q3, Q4, R10, R11, R12, R13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
