File: Eagle/doogie_bottom_board.brd (EAGLE design)
At the start: 239.3 x 151.4 mm, 31 parts, among them Q1 TEFT4300, Q2 TEFT4300, Q3 TEFT4300, Q4 TEFT4300, T1 BC337, T2 BC337, T3 BC337

Commit message: Add first version of schematics
Parts:
- removed MOTORS: (no value), pololu:SWITCH
- removed POWER: ON/OFF, pololu:SWITCH
- removed U$2, U$3, U$4, U$5: FRAME_A4P, doogie:FRAME_A4P
- added BATTERY_HOLDER: BATTERY_HOLDER, doogie:BATTERY_HOLDER
- added J1: (no value), SparkFun-Connectors:1X12
- added J4: (no value), SparkFun-Connectors:2X3-SHROUDED
- added J5: (no value), SparkFun-Connectors:JST-2-PTH
- added Q6: IRF9530, transistor-power:TO220BV
- added S1, S2: (no value), doogie:M9040P
- J2: device SparkFun-Connectors:2X3-SHROUDED -> SparkFun-Connectors:1X12
- Q1, Q3: device maze:TEFT4300-CE -> doogie:TEFT_5MM_RA
- Q2, Q4: device maze:TEFT4300-EC -> doogie:TEFT_5MM_RA
- R10, R12, R8: value 100k -> 680R
- R11: value 2R -> 33R
- R13, R9: value 7R5 -> 47R
- U1: device doogie:TB6612FNG -> pololu:TB6612FNG
- moved J2 38.4 mm to (20.3, 15.2), turned to 90 degrees
- moved R11 36.9 mm to (26.0, 21.2), turned to 180 degrees
- moved R13 21.8 mm to (36.8, 15.9)
- moved R6 21.7 mm to (26.5, 15.9)
- moved R8 21.0 mm to (-29.1, 16.5)
- moved Q1 21.0 mm to (-35.0, 26.9)
- moved T1 21.0 mm to (-32.9, 19.8)
- moved D1 21.0 mm to (-40.1, 19.3)
- moved R4 21.0 mm to (-31.3, 24.3)
- moved R9 21.0 mm to (-40.1, 16.4)
- moved Q4 20.8 mm to (36.5, 27.4)
- moved R7 20.8 mm to (31.4, 31.3)
- moved T2 20.8 mm to (33.5, 22.1)
- moved D4 20.8 mm to (41.6, 19.8)
- moved R10 17.5 mm to (28.7, 31.4), turned to 90 degrees
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Connections:
- removed net LF_EMITTER: R8.2
- removed net LF_RECEIVER: Q1.E, R4.2
- removed net L_RECEIVER: Q2.E, R5.2
- removed net MOTORAO1: J2.2, U1.3
- removed net MOTORAO2: J2.4, U1.4
- removed net N$10: J2.6
- removed net N$17: POWER.P
- removed net RF_EMITTER: R12.2
- removed net RF_RECEIVER: Q4.E, R7.2
- removed net R_RECEIVER: Q3.E, R6.2
- removed net SIDE_EMITTER: R10.2
- removed net VCC: U1.2
- removed net VCC_1: U$1.IN+
- removed net VMOT: U1.7
- new net H-BRIDGE_!STDBY: J1.7, U1.12
- new net LEFT_FRONT_EMITTER: J1.11, R8.2
- new net LEFT_FRONT_RCVR: J1.12, Q2.E, R5.2
- new net LEFT_RCVR: J1.5, Q1.E, R4.2
- new net LEFT_RIGHT_EMITTER: J2.4
- new net LEFT_RIGHT_EMITTERS: J1.6, R10.2
- new net MOTOR_LEFT_EN1: J1.9, U1.11
- new net MOTOR_LEFT_EN2: J1.8, U1.10
- new net MOTOR_LEFT_ENCA: J1.4, J3.3
- new net MOTOR_LEFT_ENCB: J1.3, J3.2
- new net MOTOR_LEFT_O1: J3.6, U1.3
- new net MOTOR_LEFT_O2: J3.5, U1.4
- new net MOTOR_LEFT_PWM: J1.10, U1.9
- new net MOTOR_RIGHT_EN1: J2.6, U1.13
- new net MOTOR_RIGHT_EN2: J2.5, U1.14
- new net MOTOR_RIGHT_ENCA: J2.2, J4.3
- new net MOTOR_RIGHT_ENCB: J2.1, J4.2
- new net MOTOR_RIGHT_O1: J4.6, U1.6
- new net MOTOR_RIGHT_O2: J4.5, U1.5
- new net MOTOR_RIGHT_PWM: J2.7, U1.15
- new net N$8: J5.2, Q6.D
- new net N$9: Q6.S, S1.2
- new net RIGHT_FRONT_EMITTER: J2.8, R12.2
- new net RIGHT_FRONT_RCVR: J2.9, Q3.E, R6.2
- new net RIGHT_RCVR: J2.3, Q4.E, R7.2
- new net VOUT: D1.A, D2.A, D4.A, J2.10, U$1.IN+, U1.7
- net 3.3V: now also J2.12, J3.4, J4.4, U1.2; no longer D1.A, D2.A, D4.A, U$1.OUT-
- net GND: now also J1.1, J1.2, J3.1, J4.1, J5.1, Q6.G, U$1.OUT-
- net N$5: now also S2.3; no longer MOTORS.S
- net V_BATT: now also J2.11, S1.3, S2.2; no longer MOTORS.P, POWER.S
Routing:
- net LF_RECEIVER: track 1.10 -> 0.00 mm
- net LEFT_RCVR: track 0.00 -> 1.04 mm
Other:
- board text added: "MOTOR_LEFT"
- board text added: "MOTOR_RIGHT"
- board text removed: "I"
- board text removed: "LiPo 1S"
- board text removed: "O"

Commit message: Add first version of thebottom board routed
Parts:
- moved R12 48.6 mm to (31.1, 15.4), turned to 180 degrees
- moved T3 42.7 mm to (35.6, 20.8)
- moved T2 41.0 mm to (0.00, 45.7)
- moved R10 41.0 mm to (-9.65, 45.7), turned to 180 degrees
- moved R6 32.1 mm to (21.0, 47.5), turned to 210 degrees
- moved R11 29.5 mm to (9.65, 45.7), turned to 0 degrees
- moved R7 9.59 mm to (31.1, 21.7), turned to 90 degrees
- moved R13 4.22 mm to (41.0, 15.4)
- moved S1 3.15 mm to (42.2, -27.4)
- moved S2 2.98 mm to (-42.2, -27.4)
- moved T1 2.86 mm to (-35.6, 20.8)
- moved J2 2.80 mm to (23.1, 15.4)
- moved R4 2.63 mm to (-31.1, 21.7), turned to 90 degrees
- moved R5 2.33 mm to (-21.0, 47.5), turned to 330 degrees
- moved R8 2.27 mm to (-31.1, 15.4)
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Connections:
- net VOUT renamed 6V
- removed net GND: J1.1, J1.2, J3.1, J4.1, J5.1, Q6.G, R4.1, R5.1, R6.1, R7.1, T1.1, T2.1, T3.1, U$1.IN-, U$1.OUT-, U1.1, U1.16, U1.8
- removed net LEFT_FRONT_EMITTER: J1.11, R8.2
- removed net LEFT_RIGHT_EMITTER: J2.4
- removed net LEFT_RIGHT_EMITTERS: J1.6, R10.2
- removed net RIGHT_FRONT_EMITTER: J2.8, R12.2
- new net FILLING_POLYGON: J1.10, J1.2, J2.8, J3.1, J4.1, J5.1, Q6.G, R4.1, R5.1, R6.1, R7.1, T1.1, T2.1, T3.1, U$1.IN-, U$1.OUT-, U1.1, U1.16, U1.8
- new net FRONT_EMITTERS_CTRL: J1.11, R10.2
- new net LEFT_EMITTER_CTRL: J1.1, R8.2
- new net RIGHT_EMITTER_CTRL: J2.3, R12.2
- net H-BRIDGE_!STDBY: now also J1.9; no longer J1.7
- net MOTOR_LEFT_EN1: now also J1.8; no longer J1.9
- net MOTOR_LEFT_EN2: now also J1.7; no longer J1.8
- net MOTOR_LEFT_ENCA: now also J1.3; no longer J1.4
- net MOTOR_LEFT_ENCB: now also J1.4; no longer J1.3
- net MOTOR_LEFT_PWM: now also J1.6; no longer J1.10
- net MOTOR_RIGHT_EN1: now also J2.7; no longer J2.6
- net MOTOR_RIGHT_EN2: now also J2.6; no longer J2.5
- net MOTOR_RIGHT_PWM: now also J2.5; no longer J2.7
- net RIGHT_RCVR: now also J2.4; no longer J2.3
Routing:
- net 6V: track 0.00 -> 330.5 mm, vias 0 -> 2
- net 3.3V: track 0.00 -> 277.6 mm
- net V_BATT: track 0.00 -> 183.3 mm
- net N$5: track 0.00 -> 78.9 mm
- net MOTOR_RIGHT_ENCB: track 0.00 -> 51.5 mm
- net N$9: track 0.00 -> 50.2 mm
- net MOTOR_RIGHT_O2: track 0.00 -> 48.4 mm
- net MOTOR_RIGHT_ENCA: track 0.00 -> 44.2 mm
- net MOTOR_LEFT_ENCA: track 0.00 -> 43.0 mm
- net MOTOR_RIGHT_O1: track 0.00 -> 38.0 mm
- net MOTOR_LEFT_ENCB: track 0.00 -> 35.3 mm
- net H-BRIDGE_!STDBY: track 0.00 -> 32.2 mm
- net MOTOR_LEFT_O2: track 0.00 -> 29.9 mm
- net MOTOR_LEFT_EN1: track 0.00 -> 27.2 mm
- net MOTOR_RIGHT_EN1: track 0.00 -> 27.1 mm
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- added copper zone on layer 1, net FILLING_POLYGON
- added copper zone on layer 16, net FILLING_POLYGON
- removed copper zone on layer 16, net GND
Other:
- board text added: "DOOGIE MOUSE V1.0"
- board text removed: "TON-BOT V1.1"

Commit message: Route bottom board
Parts:
- D1: device maze:SFH4545-AK -> doogie:SFH4545-AK
- D2, D3: device maze:SFH4545-KA -> doogie:SFH4545-AK
- D4: value SFH4545KA -> SFH4545; device maze:SFH4545-KA -> doogie:SFH4545-AK
Routing:
- net N$20: track 16.9 -> 13.4 mm
- net N$16: track 6.55 -> 3.99 mm
- net N$14: track 8.89 -> 6.35 mm
- net 6V: track 330.5 -> 328.1 mm
Other:
- board size 239.3 x 151.4 mm -> 92.9 x 98 mm
- board text added: "+"
- board text added: "-"
- board text added: "/home/menezes/Pictures/power-button-off.bmp"
- board text added: "OFF"
- board text added: "ON"

Commit message: Make top board routing sketch
Other:
- board text added: "DOOGIE MOUSE V1.0 by Doogie Team Licensed under CERN OHL v.1.2. http://ohwr.org/cernohl"
- board text removed: "TON-BOT V1.1 by IOTON Technology. Licensed under CERN OHL v.1.2. http://ohwr.org/cernohl"
Changed lines of the file:
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@@
 <layer number="16" name="Bottom" color="1" fill="1" visible="no" active="yes"/>
 <layer number="17" name="Pads" color="2" fill="1" visible="yes" active="yes"/>
-<layer number="18" name="Vias" color="14" fill="1" visible="no" active="yes"/>
-<layer number="19" name="Unrouted" color="6" fill="1" visible="no" active="yes"/>
+<layer number="18" name="Vias" color="14" fill="1" visible="yes" active="yes"/>
+<layer number="19" name="Unrouted" color="6" fill="1" visible="yes" active="yes"/>
 <layer number="20" name="Dimension" color="15" fill="1" visible="yes" active="yes"/>
-<layer number="21" name="tPlace" color="7" fill="1" visible="no" active="yes"/>
+<layer number="21" name="tPlace" color="7" fill="1" visible="yes" active="yes"/>
 <layer number="22" name="bPlace" color="7" fill="1" visible="no" active="yes"/>
-<layer number="23" name="tOrigins" color="15" fill="1" visible="no" active="yes"/>
+<layer number="23" name="tOrigins" color="15" fill="1" visible="yes" active="yes"/>
 <layer number="24" name="bOrigins" color="15" fill="1" visible="no" active="yes"/>
-<layer number="25" name="tNames" color="7" fill="1" visible="no" active="yes"/>
+<layer number="25" name="tNames" color="7" fill="1" visible="yes" active="yes"/>
 <layer number="26" name="bNames" color="7" fill="1" visible="no" active="yes"/>
 <layer number="27" name="tValues" color="7" fill="1" visible="no" active="yes"/>
 <layer number="28" name="bValues" color="7" fill="1" visible="no" active="yes"/>
-<layer number="29" name="tStop" color="7" fill="3" visible="yes" active="yes"/>
+<layer number="29" name="tStop" color="7" fill="3" visible="no" active="yes"/>
 <layer number="30" name="bStop" color="7" fill="6" visible="no" active="yes"/>
 <layer number="31" name="tCream" color="7" fill="4" visible="no" active="yes"/>
@@
 <layer number="37" name="tTest" color="7" fill="1" visible="no" active="yes"/>
 <layer number="38" name="bTest" color="7" fill="1" visible="no" active="yes"/>
-<layer number="39" name="tKeepout" color="4" fill="11" visible="no" active="yes"/>
+<layer number="39" name="tKeepout" color="4" fill="11" visible="yes" active="yes"/>
 <layer number="40" name="bKeepout" color="1" fill="11" visible="no" active="yes"/>
-<layer number="41" name="tRestrict" color="4" fill="10" visible="no" active="yes"/>
+<layer number="41" name="tRestrict" color="4" fill="10" visible="yes" active="yes"/>
 <layer number="42" name="bRestrict" color="1" fill="10" visible="no" active="yes"/>
 <layer number="43" name="vRestrict" color="2" fill="10" visible="no" active="yes"/>
@@
 <layer number="49" name="Reference" color="7" fill="1" visible="no" active="yes"/>
 <layer number="50" name="dxf" color="7" fill="1" visible="no" active="no"/>
-<layer number="51" name="tDocu" color="14" fill="1" visible="no" active="yes"/>
+<layer number="51" name="tDocu" color="14" fill="1" visible="yes" active="yes"/>
 <layer number="52" name="bDocu" color="6" fill="1" visible="no" active="yes"/>
 <layer number="53" name="tGND_GNDA" color="7" fill="9" visible="no" active="no"/>
@@
 <circle x="32.9825" y="-9.47" radius="1.419903125" width="0.3048" layer="42"/>
 <rectangle x1="-6.6675" y1="49.53" x2="-6.0325" y2="50.165" layer="42"/>
-<text x="-9.7155" y="65.024" size="1.27" layer="51">TON-BOT V1.1 by IOTON Technology.
+<text x="-9.7155" y="65.024" size="1.27" layer="51">DOOGIE MOUSE V1.0 by Doogie Team
 Licensed under CERN OHL v.1.2.
 http://ohwr.org/cernohl</text>
