File: Eagle/doogie_top_board.sch (EAGLE design)
At the start: 26 parts, among them U1 GY-521MPU6050

Commit message: Add first version of schematics
Parts:
- removed OK1, OK2, OK3, OK4, OK5, OK6, OK7: PC817, optocoupler:PC817
- removed R10, R11, R12, R13, R14, R7, R8, R9: (no value), rcl:R-EU_0204/7
- added BUZZER: F/TMB, buzzer:F/TMB
- added D1, D2: GREEN, SparkFun-LED:LED3MM
- added D3: 1N4004, adafruit:1N4004
- added K1: G5L, relay:G5L
- added S1, S2: MOMENTARY-SWITCH-SPST-PTH-6.0MM, SparkFun-Switches:MOMENTARY-SWITCH-SPST-PTH-6.0MM
- added T1, T2: BC337, transistor:BC337
- added U2: U1V10F5, pololu:U1V10F5
- J1, J2: device SparkFun-Connectors:CONN_10" -> SparkFun-Connectors:CONN_12
- R1: value (none) -> 750R
- R2: value (none) -> 390R
- R3: value (none) -> 820R
- R4: value (none) -> 680R
- R5, R6: value (none) -> 10k
Connections:
- removed net GPIO_H-BRIDGE_!STDBY: R4.1
- removed net GPIO_MOTOR_LEFT_EN1: R2.1
- removed net GPIO_MOTOR_LEFT_EN2: R3.1
- removed net GPIO_MOTOR_LEFT_PWM: R1.1
- removed net GPIO_MOTOR_RIGHT_EN1: R6.1
- removed net GPIO_MOTOR_RIGHT_EN2: R7.1
- removed net GPIO_MOTOR_RIGHT_PWM: R5.1
- removed net VCC: R10.2, R11.2, R12.2, R13.2, R14.2, R8.2, R9.2
- new net 5V: BUZZER.+, D3.C, K11.1, U$2.5V0@1, U$2.5V0@2, U2.VOUT
- new net ADC_A0_CHANNEL: K12.P, U$3.A0
- new net BATT_MONITORING_EN: U$2.GPIO11/SCLK
- new net BUZZER_CTRL: R1.1, R4.1, U$2.GPIO10/MOSI
- new net GND@7: U$2.GND@4, U$2.GND@5, U$2.GND@6, U$2.GND@7, U$2.GND@8
- new net LEFT_RCVR_EN: U$2.GPIO9/MISO
- new net N$8: R4.2, T2.B
- new net N$9: K12.S, R5.1, R6.2
- new net VOUT: J2.10, R3.2
- net 3.3V: now also J2.12; no longer OK1.EMIT, OK2.EMIT, OK3.EMIT, OK4.EMIT, OK5.EMIT, OK6.EMIT, OK7.EMIT
- net GND: now also D1.C, D2.C, J1.1, J1.2, R6.1, S1.1, S2.1, T1.E, T2.E, U$2.GND@1, U$2.GND@2, U$2.GND@3, U2.GND; no longer OK1.C, OK2.C, OK3.C, OK4.C, OK5.C, OK6.C, OK7.C
- net H-BRIDGE_!STDBY: now also J1.7, U$2.GPIO17/GEN0; no longer J1.6, OK4.COL, R11.1
- net LEFT_FRONT_EMITTER: now also J1.11, U$2.GPIO22/GEN3; no longer J1.2
- net LEFT_FRONT_RCVR: now also J1.12; no longer J1.1
- net LEFT_RCVR: now also J1.5, K12.O; no longer J1.8, U$3.A0
- net LEFT_RIGHT_EMITTER: now also J1.6, J2.4, U$2.RXD0/GPIO15; no longer J1.7, J2.7
- net MOTOR_LEFT_EN1: now also J1.9, U$2.GPIO27/GEN2; no longer J1.4, OK2.COL, R9.1
- net MOTOR_LEFT_EN2: now also J1.8, U$2.GPIO18; no longer J1.5, OK3.COL, R10.1
- net MOTOR_LEFT_ENCA: now also J1.4, U$2.TXD0/GPIO14; no longer J1.9
- net MOTOR_LEFT_ENCB: now also J1.3, U$2.GPIO4/GCKL; no longer J1.10
- net MOTOR_LEFT_PWM: now also J1.10, U$2.GPIO19; no longer J1.3, OK1.COL, R8.1
- net MOTOR_RIGHT_EN1: now also J2.6, U$2.GPIO16; no longer J2.4, OK6.COL, R13.1
- net MOTOR_RIGHT_EN2: now also U$2.GPIO26; no longer OK7.COL, R14.1
- net MOTOR_RIGHT_ENCA: now also J2.2, U$2.GPIO20; no longer J2.9
- net MOTOR_RIGHT_ENCB: now also J2.1, U$2.GPIO21; no longer J2.10
- net MOTOR_RIGHT_PWM: now also J2.7, U$2.GPIO12; no longer J2.3, OK5.COL, R12.1
- net N$1: now also BUZZER.-, T1.C; no longer OK6.A, R6.2
- net N$2: now also R1.2, T1.B; no longer OK7.A, R7.2
- net N$3: now also S2.2, U$2.GPIO13; no longer OK5.A, R5.2
- net N$4: now also S1.2, U$2.GPIO6; no longer OK4.A, R4.2
- net N$5: now also D1.A, R2.1; no longer OK2.A, R2.2
- net N$6: now also D2.A, R3.1; no longer OK3.A, R3.2
- net N$7: now also D3.A, K11.2, T2.C; no longer OK1.A, R1.2
- net RIGHT_FRONT_EMITTER: now also J2.8, U$2.ID_SC; no longer J2.2
- net RIGHT_FRONT_RCVR: now also J2.9; no longer J2.1
- net RIGHT_RCVR: now also J2.3; no longer J2.8
- net V_BATT: now also J2.11, R2.2, R5.2, U2.VIN; no longer U$2.5V0@1, U$2.5V0@2
Other:
- note added: "Buttons to control the robot"

Commit message: Route bottom board
Parts:
- removed D3: 1N4004, adafruit:1N4004
- removed K1: G5L, relay:G5L
- removed R4: 680R, rcl:R-EU_0204/7
- removed T2: BC337, transistor:BC337
- added U3: 74HC4051_SPARKFUN, doogie:74HC4051_SPARKFUN
Connections:
- net LEFT_FRONT_EMITTER renamed FRONT_EMITTERS_CTRL
- removed net BATT_MONITORING_EN: U$2.GPIO11/SCLK
- removed net LEFT_RCVR_EN: U$2.GPIO9/MISO
- removed net LEFT_RIGHT_EMITTER: J1.6, J2.4, U$2.RXD0/GPIO15
- removed net N$7: D3.A, K11.2, T2.C
- removed net N$8: R4.2, T2.B
- removed net RIGHT_FRONT_EMITTER: J2.8, U$2.ID_SC
- new net ADC_A0_CHANNEL_CTRL: U$2.GPIO9/MISO, U3.S0
- new net LEFT_EMITTER_CTRL: J1.1, U$2.RXD0/GPIO15
- new net RIGHT_EMITTER_CTRL: J2.3, U$2.ID_SC
- net 3.3V: now also U3.VCC
- net 5V: no longer D3.C, K11.1
- net ADC_A0_CHANNEL: now also U3.Z; no longer K12.P
- net BUZZER_CTRL: no longer R4.1
- net GND: now also J1.6, U3.GND, U3.S1, U3.S2, U3.VEE; no longer J1.1, T2.E
- net LEFT_RCVR: now also U3.Y0; no longer K12.O
- net N$9: now also U3.Y1; no longer K12.S
- net RIGHT_RCVR: now also J2.4; no longer J2.3
Other:
- moved on the sheet: R5, R6

Commit message: Make top board routing sketch
Parts:
- added D3: 1N4004, diode:1N4004
- U$2: device RPI-Zero:RPI-ZERO -> doogie:RPI-ZERO
Connections:
- removed net GND@7: U$2.GND@4, U$2.GND@5, U$2.GND@6, U$2.GND@7, U$2.GND@8
- net 5V: now also D3.C
- net GND: now also J1.10, J2.8, S1.2, S2.2, U$2.GND@4, U$2.GND@5, U$2.GND@6, U$2.GND@7, U$2.GND@8; no longer J1.6, S1.1, S2.1
- net H-BRIDGE_!STDBY: now also J1.9, U$2.GPIO27/GEN2; no longer J1.7, U$2.GPIO17/GEN0
- net LEFT_EMITTER_CTRL: now also U$2.GPIO4/GCKL; no longer U$2.RXD0/GPIO15
- net MOTOR_LEFT_EN1: now also J1.8, U$2.GPIO18; no longer J1.9, U$2.GPIO27/GEN2
- net MOTOR_LEFT_EN2: now also J1.7, U$2.GPIO17/GEN0; no longer J1.8, U$2.GPIO18
- net MOTOR_LEFT_ENCA: now also J1.3; no longer J1.4
- net MOTOR_LEFT_ENCB: now also J1.4, U$2.RXD0/GPIO15; no longer J1.3, U$2.GPIO4/GCKL
- net MOTOR_LEFT_PWM: now also J1.6; no longer J1.10
- net MOTOR_RIGHT_EN1: now also J2.7, U$2.GPIO5; no longer J2.6, U$2.GPIO16
- net MOTOR_RIGHT_EN2: now also J2.6, U$2.GPIO6; no longer J2.5, U$2.GPIO26
- net MOTOR_RIGHT_ENCA: now also U$2.GPIO16; no longer U$2.GPIO20
- net MOTOR_RIGHT_ENCB: now also U$2.GPIO20; no longer U$2.GPIO21
- net MOTOR_RIGHT_PWM: now also J2.5; no longer J2.7
- net N$1: now also D3.A
- net N$3: now also S2.1, U$2.GPIO26; no longer S2.2, U$2.GPIO13
- net N$4: now also S1.1, U$2.GPIO21; no longer S1.2, U$2.GPIO6
- net RIGHT_EMITTER_CTRL: now also U$2.GPIO13; no longer U$2.ID_SC
Other:
- note removed: "Buttons to control the robot"
- moved on the sheet: S1, S2, U2

Commit message: Add first step of top board routing
Parts:
- U$3: device diy-modules:ADC-4CH-ADS1115 -> doogie:ADC-4CH-ADS1115
Connections:
- removed net ADC_A0_CHANNEL: U$3.A0, U3.Z
- removed net ADC_A0_CHANNEL_CTRL: U$2.GPIO9/MISO, U3.S0
- new net ADC_A1_CHANNEL: U$3.A1, U3.Z
- new net ADC_A1_CHANNEL_CTRL: U$2.GPIO11/SCLK, U3.S0
- net H-BRIDGE_!STDBY: now also U$2.GEN4/GPIO23; no longer U$2.GPIO27/GEN2
- net LEFT_FRONT_RCVR: now also U$3.A0; no longer U$3.A1
- net MOTOR_LEFT_EN1: now also U$2.GPIO27/GEN2; no longer U$2.GPIO18
- net MOTOR_LEFT_PWM: now also U$2.GPIO18; no longer U$2.GPIO19
- net MOTOR_RIGHT_EN1: now also U$2.GPIO6; no longer U$2.GPIO5
- net MOTOR_RIGHT_EN2: now also U$2.GPIO12; no longer U$2.GPIO6
- net MOTOR_RIGHT_PWM: now also U$2.GPIO19; no longer U$2.GPIO12
Changed lines of the file:
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@@
 <setting verticaltext="up"/>
 </settings>
-<grid distance="0.1" unitdist="inch" unit="inch" style="lines" multiple="1" display="yes" altdistance="0.01" altunitdist="inch" altunit="inch"/>
+<grid distance="0.1" unitdist="inch" unit="inch" style="lines" multiple="1" display="no" altdistance="0.01" altunitdist="inch" altunit="inch"/>
 <layers>
 <layer number="1" name="Top" color="4" fill="1" visible="no" active="no"/>
@@
 <part name="U$2" library="doogie" deviceset="RPI-ZERO" device=""/>
 <part name="U1" library="gy-521" deviceset="GY-521" device="MPU6050"/>
-<part name="U$3" library="diy-modules" deviceset="ADC-4CH-ADS1115" device=""/>
+<part name="U$3" library="doogie" deviceset="ADC-4CH-ADS1115" device=""/>
 <part name="SUPPLY2" library="SparkFun-PowerSymbols" library_urn="urn:adsk.eagle:library:530" deviceset="3.3V" device=""/>
 <part name="U$4" library="doogie" deviceset="FRAME_A4P" device="">
@@
 <net name="MOTOR_RIGHT_PWM" class="0">
 <segment>
+<label x="205.74" y="78.74" size="1.27" layer="95" xref="yes"/>
+<pinref part="J2" gate="G$1" pin="5"/>
+<wire x1="200.66" y1="78.74" x2="205.74" y2="78.74" width="0.1524" layer="91"/>
+</segment>
+<segment>
+<pinref part="U$2" gate="G$1" pin="GPIO19"/>
+<wire x1="93.98" y1="81.28" x2="83.82" y2="81.28" width="0.1524" layer="91"/>
+<label x="83.82" y="81.28" size="1.27" layer="95" rot="R180" xref="yes"/>
+</segment>
+</net>
+<net name="MOTOR_RIGHT_EN1" class="0">
+<segment>
+<label x="205.74" y="83.82" size="1.27" layer="95" xref="yes"/>
+<pinref part="J2" gate="G$1" pin="7"/>
+<wire x1="200.66" y1="83.82" x2="205.74" y2="83.82" width="0.1524" layer="91"/>
+</segment>
+<segment>
+<label x="83.82" y="86.36" size="1.27" layer="95" rot="R180" xref="yes"/>
+<pinref part="U$2" gate="G$1" pin="GPIO6"/>
+<wire x1="93.98" y1="86.36" x2="83.82" y2="86.36" width="0.1524" layer="91"/>
+</segment>
+</net>
+<net name="MOTOR_RIGHT_EN2" class="0">
+<segment>
+<label x="205.74" y="81.28" size="1.27" layer="95" xref="yes"/>
+<pinref part="J2" gate="G$1" pin="6"/>
+<wire x1="200.66" y1="81.28" x2="205.74" y2="81.28" width="0.1524" layer="91"/>
+</segment>
+<segment>
 <pinref part="U$2" gate="G$1" pin="GPIO12"/>
 <wire x1="142.24" y1="86.36" x2="152.4" y2="86.36" width="0.1524" layer="91"/>
 <label x="152.4" y="86.36" size="1.27" layer="95" xref="yes"/>
 </segment>
-<segment>
-<label x="205.74" y="78.74" size="1.27" layer="95" xref="yes"/>
-<pinref part="J2" gate="G$1" pin="5"/>
-<wire x1="200.66" y1="78.74" x2="205.74" y2="78.74" width="0.1524" layer="91"/>
-</segment>
-</net>
-<net name="MOTOR_RIGHT_EN1" class="0">
-<segment>
-<label x="205.74" y="83.82" size="1.27" layer="95" xref="yes"/>
-<pinref part="J2" gate="G$1" pin="7"/>
-<wire x1="200.66" y1="83.82" x2="205.74" y2="83.82" width="0.1524" layer="91"/>
-</segment>
-<segment>
-<pinref part="U$2" gate="G$1" pin="GPIO5"/>
-<wire x1="93.98" y1="88.9" x2="83.82" y2="88.9" width="0.1524" layer="91"/>
-<label x="83.82" y="88.9" size="1.27" layer="95" rot="R180" xref="yes"/>
-</segment>
-</net>
-<net name="MOTOR_RIGHT_EN2" class="0">
-<segment>
-<label x="205.74" y="81.28" size="1.27" layer="95" xref="yes"/>
-<pinref part="J2" gate="G$1" pin="6"/>
-<wire x1="200.66" y1="81.28" x2="205.74" y2="81.28" width="0.1524" layer="91"/>
-</segment>
-<segment>
-<pinref part="U$2" gate="G$1" pin="GPIO6"/>
-<wire x1="93.98" y1="86.36" x2="83.82" y2="86.36" width="0.1524" layer="91"/>
-<label x="83.82" y="86.36" size="1.27" layer="95" rot="R180" xref="yes"/>
-</segment>
 </net>
 <net name="MOTOR_LEFT_PWM" class="0">
-<segment>
-<pinref part="U$2" gate="G$1" pin="GPIO19"/>
-<wire x1="93.98" y1="81.28" x2="83.82" y2="81.28" width="0.1524" layer="91"/>
-<label x="83.82" y="81.28" size="1.27" layer="95" rot="R180" xref="yes"/>
-</segment>
 <segment>
 <pinref part="J1" gate="G$1" pin="6"/>
@@
 <label x="205.74" y="134.62" size="1.27" layer="95" xref="yes"/>
 </segment>
+<segment>
+<pinref part="U$2" gate="G$1" pin="GPIO18"/>
+<wire x1="142.24" y1="111.76" x2="152.4" y2="111.76" width="0.1524" layer="91"/>
+<label x="152.4" y="111.76" size="1.27" layer="95" xref="yes"/>
+</segment>
 </net>
 <net name="MOTOR_LEFT_EN1" class="0">
@@
 </segment>
 <segment>
-<pinref part="U$2" gate="G$1" pin="GPIO18"/>
-<wire x1="142.24" y1="111.76" x2="152.4" y2="111.76" width="0.1524" layer="91"/>
-<label x="152.4" y="111.76" size="1.27" layer="95" xref="yes"/>
+<pinref part="U$2" gate="G$1" pin="GPIO27/GEN2"/>
+<wire x1="93.98" y1="109.22" x2="83.82" y2="109.22" width="0.1524" layer="91"/>
+<label x="83.82" y="109.22" size="1.27" layer="95" rot="R180" xref="yes"/>
 </segment>
 </net>
@@
 </segment>
 <segment>
-<pinref part="U$2" gate="G$1" pin="GPIO27/GEN2"/>
-<wire x1="93.98" y1="109.22" x2="83.82" y2="109.22" width="0.1524" layer="91"/>
-<label x="83.82" y="109.22" size="1.27" layer="95" rot="R180" xref="yes"/>
+<pinref part="U$2" gate="G$1" pin="GEN4/GPIO23"/>
+<wire x1="142.24" y1="106.68" x2="152.4" y2="106.68" width="0.1524" layer="91"/>
+<label x="152.4" y="106.68" size="1.27" layer="95" xref="yes"/>
 </segment>
 </net>
@@
 </segment>
 </net>
-<net name="ADC_A0_CHANNEL_CTRL" class="0">
-<segment>
-<pinref part="U$2" gate="G$1" pin="GPIO9/MISO"/>
-<wire x1="93.98" y1="99.06" x2="83.82" y2="99.06" width="0.1524" layer="91"/>
-<label x="83.82" y="99.06" size="1.27" layer="95" rot="R180" xref="yes"/>
+<net name="ADC_A1_CHANNEL_CTRL" class="0">
+<segment>
+<label x="83.82" y="96.52" size="1.27" layer="95" rot="R180" xref="yes"/>
+<pinref part="U$2" gate="G$1" pin="GPIO11/SCLK"/>
+<wire x1="93.98" y1="96.52" x2="83.82" y2="96.52" width="0.1524" layer="91"/>
 </segment>
 </net>
@@
 <net name="LEFT_FRONT_RCVR" class="0">
 <segment>
-<pinref part="U$3" gate="G$1" pin="A1"/>
-<wire x1="182.88" y1="129.54" x2="172.72" y2="129.54" width="0.1524" layer="91"/>
-<label x="172.72" y="129.54" size="1.27" layer="95" rot="R180" xref="yes"/>
+<pinref part="U$3" gate="G$1" pin="A0"/>
+<wire x1="182.88" y1="132.08" x2="172.72" y2="132.08" width="0.1524" layer="91"/>
+<label x="172.72" y="132.08" size="1.27" layer="95" rot="R180" xref="yes"/>
 </segment>
 </net>
@@
 </segment>
 </net>
-<net name="ADC_A0_CHANNEL" class="0">
-<segment>
-<pinref part="U$3" gate="G$1" pin="A0"/>
-<wire x1="182.88" y1="132.08" x2="172.72" y2="132.08" width="0.1524" layer="91"/>
-<label x="172.72" y="132.08" size="1.27" layer="95" rot="R180" xref="yes"/>
-</segment>
-<segment>
-<pinref part="U3" gate="G$1" pin="Z"/>
-<wire x1="55.88" y1="60.96" x2="50.8" y2="60.96" width="0.127" layer="91"/>
-<label x="50.8" y="60.96" size="1.27" layer="95" rot="R180" xref="yes"/>
-</segment>
-</net>
 <net name="LEFT_RCVR" class="0">
 <segment>
@@
 </segment>
 </net>
-<net name="ADC_A0_CHANNEL_CTRL" class="0">
+<net name="ADC_A1_CHANNEL" class="0">
+<segment>
+<pinref part="U$3" gate="G$1" pin="A1"/>
+<wire x1="182.88" y1="129.54" x2="172.72" y2="129.54" width="0.1524" layer="91"/>
+<label x="172.72" y="129.54" size="1.27" layer="95" rot="R180" xref="yes"/>
+</segment>
+<segment>
+<pinref part="U3" gate="G$1" pin="Z"/>
+<wire x1="55.88" y1="60.96" x2="50.8" y2="60.96" width="0.127" layer="91"/>
+<label x="50.8" y="60.96" size="1.27" layer="95" rot="R180" xref="yes"/>
+</segment>
+</net>
+<net name="ADC_A1_CHANNEL_CTRL" class="0">
 <segment>
 <pinref part="U3" gate="G$1" pin="S0"/>

Commit message: Add silk
Parts:
- removed U$2: RPI-ZERO, doogie:RPI-ZERO
- added U5: 74HC4051_SPARKFUN, doogie:74HC4051_SPARKFUN
- U1: value GY-521MPU6050 -> RPI-ZERO; device gy-521:GY-521MPU6050 -> doogie:RPI-ZERO
- U3: value 74HC4051_SPARKFUN -> GY-521MPU6050; device doogie:74HC4051_SPARKFUN -> doogie:GY-521MPU6050
- renumbered U$3 to U4
Connections:
- net 3.3V: now also U1.3V3@1, U1.3V3@2, U5.VCC; no longer U$2.3V3@1, U$2.3V3@2, U1.VCC
- net 5V: now also U1.5V0@1, U1.5V0@2; no longer U$2.5V0@1, U$2.5V0@2
- net ADC_A1_CHANNEL: now also U5.Z; no longer U3.Z
- net ADC_A1_CHANNEL_CTRL: now also U1.GPIO11/SCLK, U5.S0; no longer U$2.GPIO11/SCLK, U3.S0
- net BUZZER_CTRL: now also U1.GPIO10/MOSI; no longer U$2.GPIO10/MOSI
- net FRONT_EMITTERS_CTRL: now also U1.GPIO22/GEN3; no longer U$2.GPIO22/GEN3
- net GND: now also U1.GND@1, U1.GND@2, U1.GND@3, U1.GND@4, U1.GND@5, U1.GND@6, U1.GND@7, U1.GND@8, U5.GND, U5.S1, U5.S2, U5.VEE; no longer U$2.GND@1, U$2.GND@2, U$2.GND@3, U$2.GND@4, U$2.GND@5, U$2.GND@6, U$2.GND@7, U$2.GND@8, U1.GND, U3.S1, U3.S2, U3.VEE
- net H-BRIDGE_!STDBY: now also U1.GEN4/GPIO23; no longer U$2.GEN4/GPIO23
- net I2C_SCL: now also U1.GPIO3/SCL1, U3.SCL; no longer U$2.GPIO3/SCL1, U1.SCL
- net I2C_SDA: now also U1.GPIO2/SDA1, U3.SDA; no longer U$2.GPIO2/SDA1, U1.SDA
- net LEFT_EMITTER_CTRL: now also U1.GPIO4/GCKL; no longer U$2.GPIO4/GCKL
- net LEFT_RCVR: now also U5.Y0; no longer U3.Y0
- net MOTOR_LEFT_EN1: now also U1.GPIO27/GEN2; no longer U$2.GPIO27/GEN2
- net MOTOR_LEFT_EN2: now also U1.GPIO17/GEN0; no longer U$2.GPIO17/GEN0
- net MOTOR_LEFT_ENCA: now also U1.TXD0/GPIO14; no longer U$2.TXD0/GPIO14
- net MOTOR_LEFT_ENCB: now also U1.RXD0/GPIO15; no longer U$2.RXD0/GPIO15
- net MOTOR_LEFT_PWM: now also U1.GPIO18; no longer U$2.GPIO18
- net MOTOR_RIGHT_EN1: now also U1.GPIO6; no longer U$2.GPIO6
- net MOTOR_RIGHT_EN2: now also U1.GPIO12; no longer U$2.GPIO12
- net MOTOR_RIGHT_ENCA: now also U1.GPIO16; no longer U$2.GPIO16
- net MOTOR_RIGHT_ENCB: now also U1.GPIO20; no longer U$2.GPIO20
- net MOTOR_RIGHT_PWM: now also U1.GPIO19; no longer U$2.GPIO19
- net N$3: now also U1.GPIO26; no longer U$2.GPIO26
- net N$4: now also U1.GPIO21; no longer U$2.GPIO21
- net N$9: now also U5.Y1; no longer U3.Y1
- net RIGHT_EMITTER_CTRL: now also U1.GPIO13; no longer U$2.GPIO13
